File: orient_test.brd (EAGLE design)
At the start: 160 x 100 mm, 3 parts

Commit message: update
Parts:
- added R1, R2: 1.8k, resistor:0204V
- added R3: 2.2k, resistor:0204V
- added X1: 332-06, con-garry:332-06
- moved B1 14.9 mm to (80.0, 39.4)
Connections:
- removed net VCC: XR1.1
- new net +5V: R1.1, R2.1, X1.2, XR1.1
- new net N$1: OK1.1, R1.2
- new net N$2: OK1.3, R2.2
- new net N$3: OK1.5, R3.2
- new net N$4: OK1.2, X1.3, XR1.2
- new net N$5: OK1.4, X1.4, XR1.4
- new net N$6: B1.+, R3.1
- new net N$7: B1.-, OK1.6
- new net N$8: B1.AC1, X1.1
- new net N$9: B1.AC2, X1.6
- net GND: now also X1.5
Routing:
- net N$4: track 0.00 -> 66.6 mm
- net N$5: track 0.00 -> 62.6 mm
- net +5V: track 0.00 -> 55.4 mm
- net GND: track 0.00 -> 37.9 mm
- net N$8: track 0.00 -> 20.6 mm
- net N$7: track 0.00 -> 19.3 mm
- net N$9: track 0.00 -> 10.7 mm
- net N$3: track 0.00 -> 8.66 mm
- net N$2: track 0.00 -> 8.12 mm
- net N$1: track 0.00 -> 7.83 mm
- net N$6: track 0.00 -> 5.08 mm
Changed lines of the file:
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@@
 <layer number="97" name="Info" color="7" fill="1" visible="no" active="no"/>
 <layer number="98" name="Guide" color="6" fill="1" visible="no" active="no"/>
+<layer number="99" name="SpiceOrder" color="5" fill="1" visible="no" active="no"/>
 </layers>
 <board>
@@
 <param name="RoutingGrid" value="50mil"/>
 <param name="AutoGrid" value="1"/>
-<param name="Efforts" value="0"/>
+<param name="Efforts" value="2"/>
 <param name="TopRouterVariant" value="1"/>
 <param name="tpViaShape" value="round"/>
@@
 <attribute name="MPN" value="" x="41.91" y="54.61" size="1.778" layer="27" rot="R180" display="off"/>
 </element>
-<element name="B1" library="rectifier" package="2KBB-R" value="RECTIFIER-2KBB-R" x="66.04" y="34.29" rot="R270"/>
+<element name="B1" library="rectifier" package="2KBB-R" value="RECTIFIER-2KBB-R" x="80.01" y="39.37" rot="R270"/>
+<element name="R1" library="resistor" package="0204V" value="1.8k" x="81.28" y="59.69"/>
+<element name="R2" library="resistor" package="0204V" value="1.8k" x="81.28" y="55.88"/>
+<element name="R3" library="resistor" package="0204V" value="2.2k" x="81.28" y="52.07"/>
+<element name="X1" library="con-garry" package="332-06" value="332-06" x="68.58" y="33.02"/>
 </elements>
 <signals>
-<signal name="VCC">
+<signal name="N$1">
+<contactref element="OK1" pad="1"/>
+<contactref element="R1" pad="2"/>
+<wire x1="90.0684" y1="59.8932" x2="82.7532" y2="59.8932" width="0.254" layer="1"/>
+<wire x1="82.7532" y1="59.8932" x2="82.55" y2="59.69" width="0.254" layer="1"/>
+<wire x1="90.0684" y1="59.8932" x2="90.17" y2="59.69" width="0.254" layer="1"/>
+</signal>
+<signal name="N$2">
+<contactref element="OK1" pad="3"/>
+<contactref element="R2" pad="2"/>
+<wire x1="83.8962" y1="54.6354" x2="90.0684" y2="54.6354" width="0.254" layer="1"/>
+<wire x1="82.7532" y1="55.7784" x2="83.8962" y2="54.6354" width="0.254" layer="1"/>
+<wire x1="90.0684" y1="54.6354" x2="90.17" y2="54.61" width="0.254" layer="1"/>
+<wire x1="82.7532" y1="55.7784" x2="82.55" y2="55.88" width="0.254" layer="1"/>
+</signal>
+<signal name="N$3">
+<contactref element="OK1" pad="5"/>
+<contactref element="R3" pad="2"/>
+<wire x1="85.0392" y1="49.6062" x2="90.0684" y2="49.6062" width="0.254" layer="1"/>
+<wire x1="82.7532" y1="51.8922" x2="85.0392" y2="49.6062" width="0.254" layer="1"/>
+<wire x1="90.0684" y1="49.6062" x2="90.17" y2="49.53" width="0.254" layer="1"/>
+<wire x1="82.7532" y1="51.8922" x2="82.55" y2="52.07" width="0.254" layer="1"/>
+</signal>
+<signal name="N$4">
+<contactref element="X1" pad="3"/>
+<contactref element="OK1" pad="2"/>
+<contactref element="XR1" pad="2"/>
+<wire x1="51.6636" y1="54.4068" x2="50.292" y2="54.4068" width="0.254" layer="16"/>
+<wire x1="71.7804" y1="34.29" x2="68.3514" y2="37.719" width="0.254" layer="16"/>
+<wire x1="68.3514" y1="37.719" x2="51.6636" y2="54.4068" width="0.254" layer="16"/>
+<wire x1="71.7804" y1="31.5468" x2="71.7804" y2="34.29" width="0.254" layer="16"/>
+<wire x1="71.0946" y1="30.861" x2="71.7804" y2="31.5468" width="0.254" layer="16"/>
+<wire x1="69.723" y1="30.861" x2="71.0946" y2="30.861" width="0.254" layer="16"/>
+<wire x1="68.58" y1="32.004" x2="69.723" y2="30.861" width="0.254" layer="16"/>
+<wire x1="50.292" y1="54.4068" x2="50.165" y2="54.61" width="0.254" layer="16"/>
+<wire x1="68.58" y1="32.004" x2="68.58" y2="32.02" width="0.254" layer="16"/>
+<wire x1="89.154" y1="57.15" x2="90.17" y2="57.15" width="0.254" layer="16"/>
+<wire x1="80.2386" y1="48.2346" x2="89.154" y2="57.15" width="0.254" layer="16"/>
+<wire x1="78.867" y1="48.2346" x2="80.2386" y2="48.2346" width="0.254" layer="16"/>
+<wire x1="68.3514" y1="37.719" x2="78.867" y2="48.2346" width="0.254" layer="16"/>
+</signal>
+<signal name="N$5">
+<contactref element="X1" pad="4"/>
+<contactref element="OK1" pad="4"/>
+<contactref element="XR1" pad="4"/>
+<wire x1="47.7774" y1="53.0352" x2="47.7774" y2="54.4068" width="0.254" layer="16"/>
+<wire x1="65.6082" y1="35.2044" x2="47.7774" y2="53.0352" width="0.254" layer="16"/>
+<wire x1="67.437" y1="35.2044" x2="65.6082" y2="35.2044" width="0.254" layer="16"/>
+<wire x1="68.58" y1="34.0614" x2="67.437" y2="35.2044" width="0.254" layer="16"/>
+<wire x1="47.7774" y1="54.4068" x2="47.625" y2="54.61" width="0.254" layer="16"/>
+<wire x1="68.58" y1="34.0614" x2="68.58" y2="34.02" width="0.254" layer="16"/>
+<wire x1="90.297" y1="50.9778" x2="90.297" y2="51.8922" width="0.254" layer="1"/>
+<wire x1="91.2114" y1="50.0634" x2="90.297" y2="50.9778" width="0.254" layer="1"/>
+<wire x1="91.2114" y1="49.149" x2="91.2114" y2="50.0634" width="0.254" layer="1"/>
+<wire x1="90.0684" y1="48.006" x2="91.2114" y2="49.149" width="0.254" layer="1"/>
+<wire x1="83.439" y1="48.006" x2="90.0684" y2="48.006" width="0.254" layer="1"/>
+<wire x1="70.6374" y1="35.2044" x2="83.439" y2="48.006" width="0.254" layer="1"/>
+<wire x1="69.723" y1="35.2044" x2="70.6374" y2="35.2044" width="0.254" layer="1"/>
+<wire x1="68.58" y1="34.0614" x2="69.723" y2="35.2044" width="0.254" layer="1"/>
+<wire x1="90.297" y1="51.8922" x2="90.17" y2="52.07" width="0.254" layer="1"/>
+<wire x1="68.58" y1="34.0614" x2="68.58" y2="34.02" width="0.254" layer="1"/>
+</signal>
+<signal name="N$6">
+<contactref element="B1" pad="+"/>
+<contactref element="R3" pad="1"/>
+<wire x1="80.01" y1="46.99" x2="80.01" y2="52.07" width="0.254" layer="1"/>
+</signal>
+<signal name="N$7">
+<contactref element="B1" pad="-"/>
+<contactref element="OK1" pad="6"/>
+<wire x1="88.6968" y1="45.4914" x2="90.0684" y2="46.863" width="0.254" layer="1"/>
+<wire x1="88.4682" y1="45.4914" x2="88.6968" y2="45.4914" width="0.254" layer="1"/>
+<wire x1="82.0674" y1="39.0906" x2="88.4682" y2="45.4914" width="0.254" layer="1"/>
+<wire x1="82.0674" y1="34.0614" x2="82.0674" y2="39.0906" width="0.254" layer="1"/>
+<wire x1="80.01" y1="32.004" x2="82.0674" y2="34.0614" width="0.254" layer="1"/>
+<wire x1="90.0684" y1="46.863" x2="90.17" y2="46.99" width="0.254" layer="1"/>
+<wire x1="80.01" y1="32.004" x2="80.01" y2="31.9786" width="0.254" layer="1"/>
+</signal>
+<signal name="N$8">
+<contactref element="B1" pad="AC1"/>
+<contactref element="X1" pad="1"/>
+<wire x1="68.3514" y1="30.4038" x2="66.7512" y2="32.004" width="0.254" layer="16"/>
+<wire x1="71.3232" y1="30.4038" x2="68.3514" y2="30.4038" width="0.254" layer="16"/>
+<wire x1="77.9526" y1="37.0332" x2="71.3232" y2="30.4038" width="0.254" layer="16"/>
+<wire x1="77.9526" y1="39.7764" x2="77.9526" y2="37.0332" width="0.254" layer="16"/>
+<wire x1="80.01" y1="41.8338" x2="77.9526" y2="39.7764" width="0.254" layer="16"/>
+<wire x1="66.7512" y1="32.004" x2="66.58" y2="32.02" width="0.254" layer="16"/>
+<wire x1="80.01" y1="41.8338" x2="80.01" y2="41.9862" width="0.254" layer="16"/>
+</signal>
+<signal name="N$9">
+<contactref element="B1" pad="AC2"/>
+<contactref element="X1" pad="6"/>
+<wire x1="77.2668" y1="34.0614" x2="70.6374" y2="34.0614" width="0.254" layer="1"/>
+<wire x1="80.01" y1="36.8046" x2="77.2668" y2="34.0614" width="0.254" layer="1"/>
+<wire x1="70.6374" y1="34.0614" x2="70.58" y2="34.02" width="0.254" layer="1"/>
+<wire x1="80.01" y1="36.8046" x2="80.01" y2="36.957" width="0.254" layer="1"/>
+</signal>
+<signal name="+5V">
+<contactref element="R2" pad="1"/>
+<contactref element="R1" pad="1"/>
+<contactref element="X1" pad="2"/>
 <contactref element="XR1" pad="1"/>
+<wire x1="80.01" y1="59.69" x2="80.01" y2="55.88" width="0.254" layer="1"/>
+<wire x1="48.9204" y1="51.6636" x2="48.9204" y2="53.2638" width="0.254" layer="1"/>
+<wire x1="66.5226" y1="34.0614" x2="62.4078" y2="38.1762" width="0.254" layer="1"/>
+<wire x1="62.4078" y1="38.1762" x2="48.9204" y2="51.6636" width="0.254" layer="1"/>
+<wire x1="48.9204" y1="53.2638" x2="48.895" y2="53.34" width="0.254" layer="1"/>
+<wire x1="66.5226" y1="34.0614" x2="66.58" y2="34.02" width="0.254" layer="1"/>
+<wire x1="62.4078" y1="38.1762" x2="80.01" y2="55.7784" width="0.254" layer="1"/>
+<wire x1="80.01" y1="55.7784" x2="80.01" y2="55.88" width="0.254" layer="1"/>
 </signal>
 <signal name="GND">
+<contactref element="X1" pad="5"/>
 <contactref element="XR1" pad="3"/>
+<wire x1="48.6918" y1="54.4068" x2="48.6918" y2="55.7784" width="0.254" layer="1"/>
+<wire x1="48.006" y1="53.721" x2="48.6918" y2="54.4068" width="0.254" layer="1"/>
+<wire x1="48.006" y1="48.9204" x2="48.006" y2="53.721" width="0.254" layer="1"/>
+<wire x1="66.0654" y1="30.861" x2="48.006" y2="48.9204" width="0.254" layer="1"/>
+<wire x1="69.2658" y1="30.861" x2="66.0654" y2="30.861" width="0.254" layer="1"/>
+<wire x1="70.4088" y1="32.004" x2="69.2658" y2="30.861" width="0.254" layer="1"/>
+<wire x1="48.6918" y1="55.7784" x2="48.895" y2="55.88" width="0.254" layer="1"/>
+<wire x1="70.4088" y1="32.004" x2="70.58" y2="32.02" width="0.254" layer="1"/>
 </signal>
 </signals>
