File: orient_test.sch (EAGLE design)
At the start: 3 parts

Commit message: update
Parts:
- added R1, R2: 1.8k, resistor:R-US_0204/2V
- added R3: 2.2k, resistor:R-US_0204/2V
- added X1: 332-06, con-garry:332-06
Connections:
- new net +5V: R1.1, R2.1, X1-2.S, XR1.VCC
- new net GND: X1-5.S, XR1.GND
- new net N$1: OK1A.A, R1.2
- new net N$2: OK1B.A, R2.2
- new net N$3: OK1C.A, R3.2
- new net N$4: OK1A.C, X1-3.S, XR1.DA
- new net N$5: OK1B.C, X1-4.S, XR1.DB
- new net N$6: B1.+, R3.1
- new net N$7: B1.-, OK1C.C
- new net N$8: B1.AC1, X1-1.S
- new net N$9: B1.AC2, X1-6.S
Changed lines of the file:
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@@
 <layer number="97" name="Info" color="7" fill="1" visible="yes" active="yes"/>
 <layer number="98" name="Guide" color="6" fill="1" visible="yes" active="yes"/>
+<layer number="99" name="SpiceOrder" color="5" fill="1" visible="yes" active="yes"/>
 </layers>
 <schematic xreflabel="%F%N/%S.%C%R" xrefpart="/%S.%C%R">
@@
 <part name="XR1" library="opto-honeywell" deviceset="GFD1300550" device=""/>
 <part name="B1" library="rectifier" deviceset="RECTIFIER-" device="2KBB-R"/>
+<part name="R1" library="resistor" deviceset="R-US_" device="0204/2V" value="1.8k"/>
+<part name="R2" library="resistor" deviceset="R-US_" device="0204/2V" value="1.8k"/>
+<part name="R3" library="resistor" deviceset="R-US_" device="0204/2V" value="2.2k"/>
+<part name="X1" library="con-garry" deviceset="332-06" device=""/>
+<part name="P+1" library="supply1" deviceset="+5V" device=""/>
+<part name="GND1" library="supply1" deviceset="GND" device=""/>
 </parts>
 <sheets>
@@
 <instance part="XR1" gate="G$1" x="12.7" y="58.42"/>
 <instance part="B1" gate="G$1" x="15.24" y="35.56"/>
+<instance part="R1" gate="G$1" x="53.34" y="78.74"/>
+<instance part="R2" gate="G$1" x="53.34" y="63.5"/>
+<instance part="R3" gate="G$1" x="53.34" y="48.26"/>
+<instance part="X1" gate="-1" x="12.7" y="78.74"/>
+<instance part="X1" gate="-2" x="33.02" y="78.74"/>
+<instance part="X1" gate="-3" x="12.7" y="76.2"/>
+<instance part="X1" gate="-4" x="33.02" y="76.2"/>
+<instance part="X1" gate="-5" x="12.7" y="73.66"/>
+<instance part="X1" gate="-6" x="33.02" y="73.66"/>
+<instance part="P+1" gate="1" x="22.86" y="71.12"/>
+<instance part="GND1" gate="1" x="-5.08" y="48.26"/>
 </instances>
 <busses>
 </busses>
 <nets>
+<net name="N$1" class="0">
+<segment>
+<pinref part="OK1" gate="A" pin="A"/>
+<pinref part="R1" gate="G$1" pin="2"/>
+<junction x="58.42" y="78.74"/>
+</segment>
+</net>
+<net name="N$2" class="0">
+<segment>
+<pinref part="OK1" gate="B" pin="A"/>
+<pinref part="R2" gate="G$1" pin="2"/>
+<junction x="58.42" y="63.5"/>
+</segment>
+</net>
+<net name="N$3" class="0">
+<segment>
+<pinref part="OK1" gate="C" pin="A"/>
+<pinref part="R3" gate="G$1" pin="2"/>
+<junction x="58.42" y="48.26"/>
+</segment>
+</net>
+<net name="N$4" class="0">
+<segment>
+<pinref part="X1" gate="-3" pin="S"/>
+<wire x1="10.16" y1="76.2" x2="0" y2="76.2" width="0.1524" layer="91"/>
+<wire x1="0" y1="76.2" x2="0" y2="83.82" width="0.1524" layer="91"/>
+<wire x1="0" y1="83.82" x2="43.18" y2="83.82" width="0.1524" layer="91"/>
+<wire x1="43.18" y1="83.82" x2="43.18" y2="73.66" width="0.1524" layer="91"/>
+<pinref part="OK1" gate="A" pin="C"/>
+<wire x1="43.18" y1="73.66" x2="58.42" y2="73.66" width="0.1524" layer="91"/>
+<junction x="58.42" y="73.66"/>
+<junction x="10.16" y="76.2"/>
+<pinref part="XR1" gate="G$1" pin="DA"/>
+<wire x1="25.4" y1="58.42" x2="25.4" y2="66.04" width="0.1524" layer="91"/>
+<wire x1="25.4" y1="66.04" x2="43.18" y2="66.04" width="0.1524" layer="91"/>
+<wire x1="43.18" y1="66.04" x2="43.18" y2="73.66" width="0.1524" layer="91"/>
+<junction x="43.18" y="73.66"/>
+<junction x="25.4" y="58.42"/>
+</segment>
+</net>
+<net name="N$5" class="0">
+<segment>
+<pinref part="X1" gate="-4" pin="S"/>
+<wire x1="30.48" y1="76.2" x2="27.94" y2="76.2" width="0.1524" layer="91"/>
+<wire x1="27.94" y1="76.2" x2="27.94" y2="58.42" width="0.1524" layer="91"/>
+<pinref part="OK1" gate="B" pin="C"/>
+<wire x1="27.94" y1="58.42" x2="58.42" y2="58.42" width="0.1524" layer="91"/>
+<junction x="58.42" y="58.42"/>
+<junction x="30.48" y="76.2"/>
+<pinref part="XR1" gate="G$1" pin="DB"/>
+<wire x1="25.4" y1="55.88" x2="27.94" y2="55.88" width="0.1524" layer="91"/>
+<wire x1="27.94" y1="55.88" x2="27.94" y2="58.42" width="0.1524" layer="91"/>
+<junction x="27.94" y="58.42"/>
+<junction x="25.4" y="55.88"/>
+</segment>
+</net>
+<net name="N$6" class="0">
+<segment>
+<pinref part="B1" gate="G$1" pin="+"/>
+<wire x1="20.32" y1="35.56" x2="40.64" y2="35.56" width="0.1524" layer="91"/>
+<wire x1="40.64" y1="35.56" x2="40.64" y2="48.26" width="0.1524" layer="91"/>
+<pinref part="R3" gate="G$1" pin="1"/>
+<wire x1="40.64" y1="48.26" x2="48.26" y2="48.26" width="0.1524" layer="91"/>
+<junction x="20.32" y="35.56"/>
+<junction x="48.26" y="48.26"/>
+</segment>
+</net>
+<net name="N$7" class="0">
+<segment>
+<pinref part="B1" gate="G$1" pin="-"/>
+<wire x1="10.16" y1="35.56" x2="7.62" y2="35.56" width="0.1524" layer="91"/>
+<wire x1="7.62" y1="35.56" x2="7.62" y2="43.18" width="0.1524" layer="91"/>
+<pinref part="OK1" gate="C" pin="C"/>
+<wire x1="7.62" y1="43.18" x2="58.42" y2="43.18" width="0.1524" layer="91"/>
+<junction x="10.16" y="35.56"/>
+<junction x="58.42" y="43.18"/>
+</segment>
+</net>
+<net name="N$8" class="0">
+<segment>
+<pinref part="B1" gate="G$1" pin="AC1"/>
+<wire x1="15.24" y1="40.64" x2="15.24" y2="45.72" width="0.1524" layer="91"/>
+<wire x1="15.24" y1="45.72" x2="5.08" y2="45.72" width="0.1524" layer="91"/>
+<wire x1="5.08" y1="45.72" x2="5.08" y2="78.74" width="0.1524" layer="91"/>
+<pinref part="X1" gate="-1" pin="S"/>
+<wire x1="5.08" y1="78.74" x2="10.16" y2="78.74" width="0.1524" layer="91"/>
+<junction x="15.24" y="40.64"/>
+<junction x="10.16" y="78.74"/>
+</segment>
+</net>
+<net name="N$9" class="0">
+<segment>
+<pinref part="B1" gate="G$1" pin="AC2"/>
+<wire x1="15.24" y1="30.48" x2="15.24" y2="27.94" width="0.1524" layer="91"/>
+<wire x1="15.24" y1="27.94" x2="2.54" y2="27.94" width="0.1524" layer="91"/>
+<wire x1="2.54" y1="27.94" x2="2.54" y2="48.26" width="0.1524" layer="91"/>
+<wire x1="2.54" y1="48.26" x2="30.48" y2="48.26" width="0.1524" layer="91"/>
+<pinref part="X1" gate="-6" pin="S"/>
+<wire x1="30.48" y1="48.26" x2="30.48" y2="73.66" width="0.1524" layer="91"/>
+<junction x="15.24" y="30.48"/>
+<junction x="30.48" y="73.66"/>
+</segment>
+</net>
+<net name="+5V" class="0">
+<segment>
+<pinref part="R2" gate="G$1" pin="1"/>
+<pinref part="R1" gate="G$1" pin="1"/>
+<wire x1="48.26" y1="63.5" x2="48.26" y2="68.58" width="0.1524" layer="91"/>
+<pinref part="X1" gate="-2" pin="S"/>
+<wire x1="48.26" y1="68.58" x2="48.26" y2="78.74" width="0.1524" layer="91"/>
+<wire x1="30.48" y1="78.74" x2="25.4" y2="78.74" width="0.1524" layer="91"/>
+<wire x1="25.4" y1="78.74" x2="25.4" y2="68.58" width="0.1524" layer="91"/>
+<wire x1="25.4" y1="68.58" x2="48.26" y2="68.58" width="0.1524" layer="91"/>
+<junction x="48.26" y="68.58"/>
+<junction x="48.26" y="63.5"/>
+<junction x="48.26" y="78.74"/>
+<junction x="30.48" y="78.74"/>
+<pinref part="XR1" gate="G$1" pin="VCC"/>
+<wire x1="22.86" y1="60.96" x2="22.86" y2="68.58" width="0.1524" layer="91"/>
+<wire x1="22.86" y1="68.58" x2="25.4" y2="68.58" width="0.1524" layer="91"/>
+<junction x="25.4" y="68.58"/>
+<junction x="22.86" y="60.96"/>
+<pinref part="P+1" gate="1" pin="+5V"/>
+<junction x="22.86" y="68.58"/>
+</segment>
+</net>
+<net name="GND" class="0">
+<segment>
+<pinref part="X1" gate="-5" pin="S"/>
+<wire x1="10.16" y1="73.66" x2="-5.08" y2="73.66" width="0.1524" layer="91"/>
+<wire x1="-5.08" y1="73.66" x2="-5.08" y2="50.8" width="0.1524" layer="91"/>
+<pinref part="XR1" gate="G$1" pin="GND"/>
+<wire x1="22.86" y1="53.34" x2="25.4" y2="53.34" width="0.1524" layer="91"/>
+<wire x1="25.4" y1="53.34" x2="25.4" y2="50.8" width="0.1524" layer="91"/>
+<wire x1="25.4" y1="50.8" x2="-5.08" y2="50.8" width="0.1524" layer="91"/>
+<junction x="10.16" y="73.66"/>
+<junction x="22.86" y="53.34"/>
+<pinref part="GND1" gate="1" pin="GND"/>
+<junction x="-5.08" y="50.8"/>
+</segment>
+</net>
 </nets>
 </sheet>
 </sheets>
+<errors>
+</errors>
 </schematic>
 </drawing>
